File: buck.kicad_sch (KiCad schematic)
At the start: 24 parts, among them IC2 LV2862YDDCR, IC2 RT6285GSP

Commit message: BOMs away
Parts:
- C1, C12: Mouser Part Number (none) -> 603-CC0603JRX70BB103
- C11: Mouser Part Number (none) -> 187-CL10B104KB85PNL
- C3: Mouser Part Number (none) -> 187-CL10C820JB81PNC
- C5, C6: Mouser Part Number (none) -> 187-CL21A226MAYNNNE
- C7, C8: Mouser Part Number (none) -> 81-GRM188R6YA475KE5D
- C8: Mouser Part Number (none) -> 81-GRM188R6YA225KA2D
- R11, R3: Mouser Part Number (none) -> 791-RMC1/16K1003FTP
- R4: Mouser Part Number (none) -> 603-AC0603FR-076K8L
- R8: Mouser Part Number (none) -> 603-RC0603FR-0756RL
- R9: Mouser Part Number (none) -> 791-RMC16K103FTP
Changed lines of the file:
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@@
+      (effects (font (size 1.27 1.27)) hide)
+    )
+    (property "Mouser Part Number" "81-GRM188R6YA475KE5D" (at 142.24 60.96 0)
       (effects (font (size 1.27 1.27)) hide)
     )
@@
       (effects (font (size 1.27 1.27)) hide)
     )
+    (property "Mouser Part Number" "187-CL10C820JB81PNC" (at 110.49 55.88 0)
+      (effects (font (size 1.27 1.27)) hide)
+    )
     (pin "1")
     (pin "2")
@@
     )
     (property "Datasheet" "~" (at 97.79 66.04 0)
+      (effects (font (size 1.27 1.27)) hide)
+    )
+    (property "Mouser Part Number" "603-AC0603FR-076K8L" (at 97.79 66.04 0)
       (effects (font (size 1.27 1.27)) hide)
     )
@@
       (effects (font (size 1.27 1.27)) hide)
     )
+    (property "Mouser Part Number" "603-CC0603JRX70BB103" (at 71.12 83.82 0)
+      (effects (font (size 1.27 1.27)) hide)
+    )
     (pin "1")
     (pin "2")
@@
     )
     (property "Datasheet" "~" (at 172.72 127 0)
+      (effects (font (size 1.27 1.27)) hide)
+    )
+    (property "Mouser Part Number" "603-RC0603FR-0756RL" (at 172.72 127 0)
       (effects (font (size 1.27 1.27)) hide)
     )
@@
       (effects (font (size 1.27 1.27)) hide)
     )
+    (property "Mouser Part Number" "81-GRM188R6YA475KE5D" (at 135.89 60.96 0)
+      (effects (font (size 1.27 1.27)) hide)
+    )
     (pin "1")
     (pin "2")
@@
     )
     (property "Datasheet" "~" (at 144.78 135.89 0)
+      (effects (font (size 1.27 1.27)) hide)
+    )
+    (property "Mouser Part Number" "603-CC0603JRX70BB103" (at 144.78 135.89 0)
       (effects (font (size 1.27 1.27)) hide)
     )
@@
       (effects (font (size 1.27 1.27)) hide)
     )
+    (property "Mouser Part Number" "187-CL21A226MAYNNNE" (at 127 93.98 0)
+      (effects (font (size 1.27 1.27)) hide)
+    )
     (pin "1")
     (pin "2")
@@
       (effects (font (size 1.27 1.27)) hide)
     )
+    (property "Mouser Part Number" "187-CL21A226MAYNNNE" (at 133.35 93.98 0)
+      (effects (font (size 1.27 1.27)) hide)
+    )
     (pin "1")
     (pin "2")
@@
       (effects (font (size 1.27 1.27)) hide)
     )
+    (property "Mouser Part Number" "791-RMC1/16K1003FTP" (at 97.79 55.88 0)
+      (effects (font (size 1.27 1.27)) hide)
+    )
     (pin "1")
     (pin "2")
@@
     )
     (property "Datasheet" "~" (at 172.72 137.16 0)
+      (effects (font (size 1.27 1.27)) hide)
+    )
+    (property "Mouser Part Number" "791-RMC16K103FTP" (at 172.72 137.16 0)
       (effects (font (size 1.27 1.27)) hide)
     )
@@
       (effects (font (size 1.27 1.27)) hide)
     )
+    (property "Mouser Part Number" "81-GRM188R6YA225KA2D" (at 100.33 138.43 0)
+      (effects (font (size 1.27 1.27)) hide)
+    )
     (pin "1")
     (pin "2")
@@
       (effects (font (size 1.27 1.27)) hide)
     )
+    (property "Mouser Part Number" "187-CL10B104KB85PNL" (at 124.46 125.73 0)
+      (effects (font (size 1.27 1.27)) hide)
+    )
     (pin "1")
     (pin "2")
@@
       (effects (font (size 1.27 1.27)) hide)
     )
+    (property "Mouser Part Number" "791-RMC1/16K1003FTP" (at 95.25 133.35 0)
+      (effects (font (size 1.27 1.27)) hide)
+    )

Commit message: Change output filtering for the +19V to 0805 (Mouser doesn't have 0603)
Parts:
- C1, C12: Mouser Part Number 603-CC0603JRX70BB103 -> (none)
- C11: Mouser Part Number 187-CL10B104KB85PNL -> (none)
- C3: Mouser Part Number 187-CL10C820JB81PNC -> (none)
- C5, C6: footprint Capacitor_SMD:C_0603_1608Metric_Pad1.08x0.95mm_HandSolder -> Capacitor_SMD:C_0805_2012Metric_Pad1.18x1.45mm_HandSolder; Mouser Part Number 187-CL21A226MAYNNNE -> (none)
- C7, C8: Mouser Part Number 81-GRM188R6YA475KE5D -> (none)
- C8: Mouser Part Number 81-GRM188R6YA225KA2D -> (none)
- R11, R3: Mouser Part Number 791-RMC1/16K1003FTP -> (none)
- R4: Mouser Part Number 603-AC0603FR-076K8L -> (none)
- R8: Mouser Part Number 603-RC0603FR-0756RL -> (none)
- R9: Mouser Part Number 791-RMC16K103FTP -> (none)
Changed lines of the file:
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@@
-      (effects (font (size 1.27 1.27)) hide)
-    )
-    (property "Mouser Part Number" "81-GRM188R6YA475KE5D" (at 142.24 60.96 0)
       (effects (font (size 1.27 1.27)) hide)
     )
@@
       (effects (font (size 1.27 1.27)) hide)
     )
-    (property "Mouser Part Number" "187-CL10C820JB81PNC" (at 110.49 55.88 0)
-      (effects (font (size 1.27 1.27)) hide)
-    )
     (pin "1")
     (pin "2")
@@
     )
     (property "Datasheet" "~" (at 97.79 66.04 0)
-      (effects (font (size 1.27 1.27)) hide)
-    )
-    (property "Mouser Part Number" "603-AC0603FR-076K8L" (at 97.79 66.04 0)
       (effects (font (size 1.27 1.27)) hide)
     )
@@
       (effects (font (size 1.27 1.27)) hide)
     )
-    (property "Mouser Part Number" "603-CC0603JRX70BB103" (at 71.12 83.82 0)
-      (effects (font (size 1.27 1.27)) hide)
-    )
     (pin "1")
     (pin "2")
@@
     )
     (property "Datasheet" "~" (at 172.72 127 0)
-      (effects (font (size 1.27 1.27)) hide)
-    )
-    (property "Mouser Part Number" "603-RC0603FR-0756RL" (at 172.72 127 0)
       (effects (font (size 1.27 1.27)) hide)
     )
@@
       (effects (font (size 1.27 1.27)) hide)
     )
-    (property "Mouser Part Number" "81-GRM188R6YA475KE5D" (at 135.89 60.96 0)
-      (effects (font (size 1.27 1.27)) hide)
-    )
     (pin "1")
     (pin "2")
@@
     )
     (property "Datasheet" "~" (at 144.78 135.89 0)
-      (effects (font (size 1.27 1.27)) hide)
-    )
-    (property "Mouser Part Number" "603-CC0603JRX70BB103" (at 144.78 135.89 0)
       (effects (font (size 1.27 1.27)) hide)
     )
@@
       (effects (font (size 1.27 1.27)) (justify left))
     )
-    (property "Footprint" "Capacitor_SMD:C_0603_1608Metric_Pad1.08x0.95mm_HandSolder" (at 126.0348 97.79 0)
+    (property "Footprint" "Capacitor_SMD:C_0805_2012Metric_Pad1.18x1.45mm_HandSolder" (at 126.0348 97.79 0)
       (effects (font (size 1.27 1.27)) hide)
     )
     (property "Datasheet" "https://www.mouser.com/datasheet/2/585/MLCC-1837944.pdf" (at 127 93.98 0)
-      (effects (font (size 1.27 1.27)) hide)
-    )
-    (property "Mouser Part Number" "187-CL21A226MAYNNNE" (at 127 93.98 0)
       (effects (font (size 1.27 1.27)) hide)
     )
@@
       (effects (font (size 1.27 1.27)) (justify left))
     )
-    (property "Footprint" "Capacitor_SMD:C_0603_1608Metric_Pad1.08x0.95mm_HandSolder" (at 134.3152 97.79 0)
+    (property "Footprint" "Capacitor_SMD:C_0805_2012Metric_Pad1.18x1.45mm_HandSolder" (at 134.3152 97.79 0)
       (effects (font (size 1.27 1.27)) hide)
     )
@@
       (effects (font (size 1.27 1.27)) hide)
     )
-    (property "Mouser Part Number" "187-CL21A226MAYNNNE" (at 133.35 93.98 0)
-      (effects (font (size 1.27 1.27)) hide)
-    )
     (pin "1")
     (pin "2")
@@
       (effects (font (size 1.27 1.27)) hide)
     )
-    (property "Mouser Part Number" "791-RMC1/16K1003FTP" (at 97.79 55.88 0)
-      (effects (font (size 1.27 1.27)) hide)
-    )
     (pin "1")
     (pin "2")
@@
     )
     (property "Datasheet" "~" (at 172.72 137.16 0)
-      (effects (font (size 1.27 1.27)) hide)
-    )
-    (property "Mouser Part Number" "791-RMC16K103FTP" (at 172.72 137.16 0)
       (effects (font (size 1.27 1.27)) hide)
     )
@@
       (effects (font (size 1.27 1.27)) hide)
     )
-    (property "Mouser Part Number" "81-GRM188R6YA225KA2D" (at 100.33 138.43 0)
-      (effects (font (size 1.27 1.27)) hide)
-    )
     (pin "1")
     (pin "2")
@@
       (effects (font (size 1.27 1.27)) hide)
     )
-    (property "Mouser Part Number" "187-CL10B104KB85PNL" (at 124.46 125.73 0)
-      (effects (font (size 1.27 1.27)) hide)
-    )
     (pin "1")
     (pin "2")
@@
       (effects (font (size 1.27 1.27)) hide)
     )
-    (property "Mouser Part Number" "791-RMC1/16K1003FTP" (at 95.25 133.35 0)
-      (effects (font (size 1.27 1.27)) hide)
-    )
